Commit message: updated joint limits of robot urdf

File: assets/urdf/ester/urdf/ester.urdf (robot description, URDF)
Before this commit: robot ester, 22 links, 21 joints
Links:
- link front_left_hip_aa_link: geometry collision mesh filename=../meshes/leg/front_hip_aa.stl scale=0.001 0.001 0.001; visual mesh filename=../meshes/leg/front_hip_aa.stl scale=0.001 0.001 0.001
- link front_left_hip_fe_link: geometry collision mesh filename=../meshes/leg/front_left_hip_fe.stl scale=0.001 0.001 0.001; visual mesh filename=../meshes/leg/front_left_hip_fe.stl scale=0.001 0.001 0.001
- link front_left_lower_leg_link: geometry collision mesh filename=../meshes/leg/front_lower_leg.stl scale=0.001 0.001 0.001; visual mesh filename=../meshes/leg/front_lower_leg.stl scale=0.001 0.001 0.001
- link front_left_upper_leg_link: geometry collision mesh filename=../meshes/leg/front_left_upper_leg.stl scale=0.001 0.001 0.001; visual mesh filename=../meshes/leg/front_left_upper_leg.stl scale=0.001 0.001 0.001
- link front_right_hip_aa_link: geometry collision mesh filename=../meshes/leg/front_hip_aa.stl scale=0.001 0.001 0.001; visual mesh filename=../meshes/leg/front_hip_aa.stl scale=0.001 0.001 0.001
- link front_right_hip_fe_link: geometry collision mesh filename=../meshes/leg/front_right_hip_fe.stl scale=0.001 0.001 0.001; visual mesh filename=../meshes/leg/front_right_hip_fe.stl scale=0.001 0.001 0.001
- link front_right_lower_leg_link: geometry collision mesh filename=../meshes/leg/front_lower_leg.stl scale=0.001 0.001 0.001; visual mesh filename=../meshes/leg/front_lower_leg.stl scale=0.001 0.001 0.001
- link front_right_upper_leg_link: geometry collision mesh filename=../meshes/leg/front_right_upper_leg.stl scale=0.001 0.001 0.001; visual mesh filename=../meshes/leg/front_right_upper_leg.stl scale=0.001 0.001 0.001
- link front_spine_pitch_link: geometry collision mesh filename=../meshes/spine/front_spine_pitch.stl scale=0.001 0.001 0.001; visual mesh filename=../meshes/spine/front_spine_pitch.stl scale=0.001 0.001 0.001
- link rear_left_hip_aa_link: geometry collision mesh filename=../meshes/leg/front_hip_aa.stl scale=0.001 0.001 0.001; visual mesh filename=../meshes/leg/front_hip_aa.stl scale=0.001 0.001 0.001
- link rear_left_hip_fe_link: geometry collision mesh filename=../meshes/leg/rear_right_hip_fe.stl scale=0.001 0.001 0.001; visual mesh filename=../meshes/leg/rear_right_hip_fe.stl scale=0.001 0.001 0.001
- link rear_left_lower_leg_link: geometry collision mesh filename=../meshes/leg/rear_lower_leg.stl scale=0.001 0.001 0.001; visual mesh filename=../meshes/leg/rear_lower_leg.stl scale=0.001 0.001 0.001
- link rear_left_upper_leg_link: geometry collision mesh filename=../meshes/leg/rear_left_upper_leg.stl scale=0.001 0.001 0.001; visual mesh filename=../meshes/leg/rear_left_upper_leg.stl scale=0.001 0.001 0.001
- link rear_right_hip_aa_link: geometry collision mesh filename=../meshes/leg/front_hip_aa.stl scale=0.001 0.001 0.001; visual mesh filename=../meshes/leg/front_hip_aa.stl scale=0.001 0.001 0.001
- link rear_right_hip_fe_link: geometry collision mesh filename=../meshes/leg/rear_left_hip_fe.stl scale=0.001 0.001 0.001; visual mesh filename=../meshes/leg/rear_left_hip_fe.stl scale=0.001 0.001 0.001
- link rear_right_lower_leg_link: geometry collision mesh filename=../meshes/leg/rear_lower_leg.stl scale=0.001 0.001 0.001; visual mesh filename=../meshes/leg/rear_lower_leg.stl scale=0.001 0.001 0.001
- link rear_right_upper_leg_link: geometry collision mesh filename=../meshes/leg/rear_right_upper_leg.stl scale=0.001 0.001 0.001; visual mesh filename=../meshes/leg/rear_right_upper_leg.stl scale=0.001 0.001 0.001
- link rear_spine_pitch_link: geometry collision mesh filename=../meshes/spine/rear_spine_pitch.stl scale=0.001 0.001 0.001; visual mesh filename=../meshes/spine/rear_spine_pitch.stl scale=0.001 0.001 0.001
- link spine_center_link: geometry collision mesh filename=../meshes/spine/spine_center.stl scale=0.001 0.001 0.001; visual mesh filename=../meshes/spine/spine_center.stl scale=0.001 0.001 0.001
Joints:
- joint front_left_hip_fe_joint: limit lower=-3.141592653589793 upper=3.141592653589793 effort=2.5 velocity=83.775 -> lower=-0.7853981633974483 upper=0.17453292519943295 effort=2.5 velocity=83.775
- joint front_left_lower_leg_joint: limit lower=-3.1415926 upper=3.1514926 effort=2.5 velocity=83.775 -> lower=-1.5707963267948966 upper=1.5707963267948966 effort=2.5 velocity=83.775
- joint front_left_upper_leg_joint: limit lower=-3.141592653589793 upper=3.141592653589793 effort=2.5 velocity=83.775 -> lower=-1.5707963267948966 upper=1.5707963267948966 effort=2.5 velocity=83.775
- joint front_right_hip_fe_joint: limit lower=-3.141592653589793 upper=3.141592653589793 effort=2.5 velocity=83.775 -> lower=-0.17453292519943295 upper=0.7853981633974483 effort=2.5 velocity=83.775
- joint front_right_lower_leg_joint: limit lower=-3.1415926 upper=3.1514926 effort=2.5 velocity=83.775 -> lower=-1.5707963267948966 upper=1.5707963267948966 effort=2.5 velocity=83.775
- joint front_right_upper_leg_joint: limit lower=-3.141592653589793 upper=3.141592653589793 effort=2.5 velocity=83.775 -> lower=-1.5707963267948966 upper=1.5707963267948966 effort=2.5 velocity=83.775
- joint front_spine_pitch_joint: limit lower=-3.141592653589793 upper=3.141592653589793 effort=2.5 velocity=83.775 -> lower=-0.2617993877991494 upper=0.2617993877991494 effort=2.5 velocity=83.775
- joint front_spine_yaw_joint: limit lower=-3.141592653589793 upper=3.141592653589793 effort=2.5 velocity=83.775 -> lower=-0.2617993877991494 upper=0.2617993877991494 effort=2.5 velocity=83.775
- joint rear_left_hip_fe_joint: limit lower=-3.141592653589793 upper=3.141592653589793 effort=2.5 velocity=83.775 -> lower=-0.7853981633974483 upper=0.17453292519943295 effort=2.5 velocity=83.775
- joint rear_left_lower_leg_joint: limit lower=-3.1415926 upper=3.1514926 effort=2.5 velocity=83.775 -> lower=-1.5707963267948966 upper=1.5707963267948966 effort=2.5 velocity=83.775
- joint rear_left_upper_leg_joint: limit lower=-3.141592653589793 upper=3.141592653589793 effort=2.5 velocity=83.775 -> lower=-1.5707963267948966 upper=1.5707963267948966 effort=2.5 velocity=83.775
- joint rear_right_hip_fe_joint: limit lower=-3.141592653589793 upper=3.141592653589793 effort=2.5 velocity=83.775 -> lower=-0.17453292519943295 upper=0.7853981633974483 effort=2.5 velocity=83.775
- joint rear_right_lower_leg_joint: limit lower=-3.1415926 upper=3.1514926 effort=2.5 velocity=83.775 -> lower=-1.5707963267948966 upper=1.5707963267948966 effort=2.5 velocity=83.775
- joint rear_right_upper_leg_joint: limit lower=-3.141592653589793 upper=3.141592653589793 effort=2.5 velocity=83.775 -> lower=-1.5707963267948966 upper=1.5707963267948966 effort=2.5 velocity=83.775
- joint rear_spine_pitch_joint: limit lower=-3.141592653589793 upper=3.141592653589793 effort=2.5 velocity=83.775 -> lower=-0.2617993877991494 upper=0.2617993877991494 effort=2.5 velocity=83.775
- joint rear_spine_yaw_joint: limit lower=-3.141592653589793 upper=3.141592653589793 effort=2.5 velocity=83.775 -> lower=-0.2617993877991494 upper=0.2617993877991494 effort=2.5 velocity=83.775

Commit message: adding foot contact sensors to see if they aid in gait growth

File: assets/urdf/ester/urdf/ester.urdf (robot description, URDF)
Before this commit: robot ester, 22 links, 21 joints
Links:
- added link front_left_foot_contact_link, mass 0.01; collision sphere radius=0.015; visual sphere radius=0.015
- added link front_right_foot_contact_link, mass 0.01; collision sphere radius=0.015; visual sphere radius=0.015
- added link rear_left_foot_contact_link, mass 0.01; collision sphere radius=0.015; visual sphere radius=0.015
- added link rear_right_foot_contact_link, mass 0.01; collision sphere radius=0.015; visual sphere radius=0.015
Joints:
- added joint front_left_foot_contact_joint: type fixed, parent front_left_lower_leg_link, child front_left_foot_contact_link, origin xyz=0 0 -0.105
- added joint front_right_foot_contact_joint: type fixed, parent front_right_lower_leg_link, child front_right_foot_contact_link, origin xyz=0 0 -0.105
- added joint rear_left_foot_contact_joint: type fixed, parent rear_left_lower_leg_link, child rear_left_foot_contact_link, origin xyz=0 0 -0.135
- added joint rear_right_foot_contact_joint: type fixed, parent rear_right_lower_leg_link, child rear_right_foot_contact_link, origin xyz=0 0 -0.135

Commit message: Adjustments to energy min reward function and increasing urdf joint torque limit to 4.45 Nm

File: assets/urdf/ester/urdf/ester.urdf (robot description, URDF)
Before this commit: robot ester, 26 links, 25 joints
Joints:
- joint front_left_hip_fe_joint: limit lower=-0.7853981633974483 upper=0.17453292519943295 effort=2.5 velocity=83.775 -> lower=-0.7853981633974483 upper=0.17453292519943295 effort=4.45 velocity=47.125
- joint front_left_lower_leg_joint: limit lower=-1.5707963267948966 upper=1.5707963267948966 effort=2.5 velocity=83.775 -> lower=-1.5707963267948966 upper=1.5707963267948966 effort=4.45 velocity=47.125
- joint front_left_upper_leg_joint: limit lower=-1.5707963267948966 upper=1.5707963267948966 effort=2.5 velocity=83.775 -> lower=-1.5707963267948966 upper=1.5707963267948966 effort=4.45 velocity=47.125
- joint front_right_hip_fe_joint: limit lower=-0.17453292519943295 upper=0.7853981633974483 effort=2.5 velocity=83.775 -> lower=-0.17453292519943295 upper=0.7853981633974483 effort=4.45 velocity=47.125
- joint front_right_lower_leg_joint: limit lower=-1.5707963267948966 upper=1.5707963267948966 effort=2.5 velocity=83.775 -> lower=-1.5707963267948966 upper=1.5707963267948966 effort=4.45 velocity=47.125
- joint front_right_upper_leg_joint: limit lower=-1.5707963267948966 upper=1.5707963267948966 effort=2.5 velocity=83.775 -> lower=-1.5707963267948966 upper=1.5707963267948966 effort=4.45 velocity=47.125
- joint front_spine_pitch_joint: limit lower=-0.2617993877991494 upper=0.2617993877991494 effort=2.5 velocity=83.775 -> lower=-0.2617993877991494 upper=0.2617993877991494 effort=4.45 velocity=47.125
- joint front_spine_yaw_joint: limit lower=-0.2617993877991494 upper=0.2617993877991494 effort=2.5 velocity=83.775 -> lower=-0.2617993877991494 upper=0.2617993877991494 effort=4.45 velocity=47.125
- joint rear_left_hip_fe_joint: limit lower=-0.7853981633974483 upper=0.17453292519943295 effort=2.5 velocity=83.775 -> lower=-0.7853981633974483 upper=0.17453292519943295 effort=4.45 velocity=47.125
- joint rear_left_lower_leg_joint: limit lower=-1.5707963267948966 upper=1.5707963267948966 effort=2.5 velocity=83.775 -> lower=-1.5707963267948966 upper=1.5707963267948966 effort=4.45 velocity=47.125
- joint rear_left_upper_leg_joint: limit lower=-1.5707963267948966 upper=1.5707963267948966 effort=2.5 velocity=83.775 -> lower=-1.5707963267948966 upper=1.5707963267948966 effort=4.45 velocity=47.125
- joint rear_right_hip_fe_joint: limit lower=-0.17453292519943295 upper=0.7853981633974483 effort=2.5 velocity=83.775 -> lower=-0.17453292519943295 upper=0.7853981633974483 effort=4.45 velocity=47.125
- joint rear_right_lower_leg_joint: limit lower=-1.5707963267948966 upper=1.5707963267948966 effort=2.5 velocity=83.775 -> lower=-1.5707963267948966 upper=1.5707963267948966 effort=4.45 velocity=47.125
- joint rear_right_upper_leg_joint: limit lower=-1.5707963267948966 upper=1.5707963267948966 effort=2.5 velocity=83.775 -> lower=-1.5707963267948966 upper=1.5707963267948966 effort=4.45 velocity=47.125
- joint rear_spine_pitch_joint: limit lower=-0.2617993877991494 upper=0.2617993877991494 effort=2.5 velocity=83.775 -> lower=-0.2617993877991494 upper=0.2617993877991494 effort=4.45 velocity=47.125
- joint rear_spine_yaw_joint: limit lower=-0.2617993877991494 upper=0.2617993877991494 effort=2.5 velocity=83.775 -> lower=-0.2617993877991494 upper=0.2617993877991494 effort=4.45 velocity=47.125

Commit message: URDF Update for 1:16 ratio joints

File: assets/urdf/ester/urdf/ester.urdf (robot description, URDF)
Before this commit: robot ester, 26 links, 25 joints
Links:
- link front_left_hip_fe_link: mass 0.153186 -> 0.139328; geometry collision mesh filename=../meshes/leg/front_hip_fe.stl scale=0.001 0.001 0.001; visual mesh filename=../meshes/leg/front_hip_fe.stl scale=0.001 0.001 0.001
- link front_left_lower_leg_link: mass 0.023609 -> 0.023961
- link front_left_upper_leg_link: mass 0.154958 -> 0.158127; geometry collision mesh filename=../meshes/leg/front_upper_leg.stl scale=0.001 0.001 0.001; visual mesh filename=../meshes/leg/front_upper_leg.stl scale=0.001 0.001 0.001
- link front_right_hip_fe_link: geometry collision mesh filename=../meshes/leg/front_hip_fe.stl scale=0.001 -0.001 0.001; visual mesh filename=../meshes/leg/front_hip_fe.stl scale=0.001 -0.001 0.001
- link front_right_lower_leg_link: mass 0.023609 -> 0.023961
- link front_right_upper_leg_link: mass 0.154958 -> 0.158127; geometry collision mesh filename=../meshes/leg/front_upper_leg.stl scale=0.001 0.001 0.001; visual mesh filename=../meshes/leg/front_upper_leg.stl scale=0.001 0.001 0.001
- link front_spine_pitch_link: mass 0.153731 -> 0.135102
- link front_spine_yaw_link: mass 0.1 -> 0.155204; geometry collision mesh filename=../meshes/spine/front_spine_yaw.stl scale=0.001 0.001 0.001; visual mesh filename=../meshes/spine/front_spine_yaw.stl scale=0.001 0.001 0.001
- link rear_left_hip_fe_link: mass 0.153223 -> 0.138767; geometry collision mesh filename=../meshes/leg/rear_hip_fe.stl scale=-0.001 0.001 0.001; visual mesh filename=../meshes/leg/rear_hip_fe.stl scale=-0.001 0.001 0.001
- link rear_left_lower_leg_link: mass 0.028708 -> 0.029071
- link rear_left_upper_leg_link: mass 0.160729 -> 0.160653; geometry collision mesh filename=../meshes/leg/rear_upper_leg.stl scale=0.001 0.001 0.001; visual mesh filename=../meshes/leg/rear_upper_leg.stl scale=0.001 0.001 0.001
- link rear_right_hip_fe_link: mass 0.158428 -> 0.138767; geometry collision mesh filename=../meshes/leg/rear_hip_fe.stl scale=0.001 0.001 0.001; visual mesh filename=../meshes/leg/rear_hip_fe.stl scale=0.001 0.001 0.001
- link rear_right_lower_leg_link: mass 0.028708 -> 0.029071
- link rear_right_upper_leg_link: mass 0.160729 -> 0.160653; geometry collision mesh filename=../meshes/leg/rear_upper_leg.stl scale=0.001 0.001 0.001; visual mesh filename=../meshes/leg/rear_upper_leg.stl scale=0.001 0.001 0.001
- link rear_spine_pitch_link: mass 0.153731 -> 0.131658
- link spine_center_link: mass 2.284352 -> 0.412971
Joints:
- joint front_left_hip_aa_joint: origin xyz=-0.0178 -0.024 -0.1065 rpy=0 0.3490658503988659 3.141592653589793 -> xyz=0.01 -0.024 -0.1065 rpy=0 0.7853981633974483 3.141592653589793
- joint front_left_hip_fe_joint: limit lower=-0.7853981633974483 upper=0.17453292519943295 effort=4.45 velocity=47.125 -> lower=-0.17453292519943295 upper=0.7853981633974483 effort=2.43 velocity=83.33333333333333; origin xyz=-0.0175 -0.0878 0 rpy=0 0 0 -> xyz=-0.083972 -0.0878 0 rpy=0 0 3.141592653589793
- joint front_left_lower_leg_joint: limit lower=-1.5707963267948966 upper=1.5707963267948966 effort=4.45 velocity=47.125 -> lower=-1.5707963267948966 upper=1.5707963267948966 effort=4.32 velocity=46.875; origin xyz=0 0.0285 -0.1232 rpy=0 0 0 -> xyz=0 0.0315 -0.1232 rpy=0 0 0
- joint front_left_upper_leg_joint: limit lower=-1.5707963267948966 upper=1.5707963267948966 effort=4.45 velocity=47.125 -> lower=-1.5707963267948966 upper=1.5707963267948966 effort=4.32 velocity=46.875; origin xyz=-0.0773 -0.013 0 rpy=0 0.3490658503988659 3.141592653589793 -> xyz=0 0.01415 0 rpy=0 0.7853981633974483 0
- joint front_right_hip_aa_joint: origin xyz=-0.0178 0.024 -0.1065 rpy=0 -0.3490658503988659 0 -> xyz=0.01 0.024 -0.1065 rpy=0 -0.7853981633974483 0
- joint front_right_hip_fe_joint: limit lower=-0.17453292519943295 upper=0.7853981633974483 effort=4.45 velocity=47.125 -> lower=-0.7853981633974483 upper=0.17453292519943295 effort=2.43 velocity=83.33333333333333; origin xyz=0.0135 -0.0878 0 rpy=0 0 3.141592653589793 -> xyz=0.083972 -0.0878 0 rpy=0 0 0
- joint front_right_lower_leg_joint: limit lower=-1.5707963267948966 upper=1.5707963267948966 effort=4.45 velocity=47.125 -> lower=-1.5707963267948966 upper=1.5707963267948966 effort=4.32 velocity=46.875; origin xyz=0 -0.0285 -0.1232 rpy=0 0 0 -> xyz=0 -0.0315 -0.1232 rpy=0 0 0
- joint front_right_upper_leg_joint: limit lower=-1.5707963267948966 upper=1.5707963267948966 effort=4.45 velocity=47.125 -> lower=-1.5707963267948966 upper=1.5707963267948966 effort=4.32 velocity=46.875; origin xyz=-0.0773 0.013 0 rpy=0 0.3490658503988659 3.141592653589793 -> xyz=0 -0.01415 0 rpy=0 0.7853981633974483 0
- joint front_spine_pitch_joint: limit lower=-0.2617993877991494 upper=0.2617993877991494 effort=4.45 velocity=47.125 -> lower=-0.2617993877991494 upper=0.2617993877991494 effort=4.32 velocity=46.875; origin xyz=0.045 0.025 -0.015 rpy=0 0 0 -> xyz=0.045 0.0 -0.015 rpy=0 0 0
- joint front_spine_yaw_joint: limit lower=-0.2617993877991494 upper=0.2617993877991494 effort=4.45 velocity=47.125 -> lower=-0.2617993877991494 upper=0.2617993877991494 effort=2.43 velocity=83.33333333333333; origin xyz=0 -0.02505 0.02115 rpy=0 0 0 -> xyz=0 0 0.02115 rpy=0 0 0
- joint rear_left_hip_aa_joint: origin xyz=-0.10425 -0.025 -0.02 rpy=0 0 3.141592653589793 -> xyz=-0.13424999999999998 -0.025 -0.02 rpy=0 0 3.141592653589793
- joint rear_left_hip_fe_joint: limit lower=-0.7853981633974483 upper=0.17453292519943295 effort=4.45 velocity=47.125 -> lower=-0.17453292519943295 upper=0.7853981633974483 effort=2.43 velocity=83.33333333333333; origin xyz=-0.0175 -0.0878 0 rpy=0 0 0 -> xyz=-0.054678 -0.0878 0 rpy=0 0 3.141592653589793
- joint rear_left_lower_leg_joint: limit lower=-1.5707963267948966 upper=1.5707963267948966 effort=4.45 velocity=47.125 -> lower=-1.5707963267948966 upper=1.5707963267948966 effort=4.32 velocity=46.875; origin xyz=0 0.0285 -0.134 rpy=0 0 0 -> xyz=0 0.0315 -0.134 rpy=0 0 0
- joint rear_left_upper_leg_joint: limit lower=-1.5707963267948966 upper=1.5707963267948966 effort=4.45 velocity=47.125 -> lower=-1.5707963267948966 upper=1.5707963267948966 effort=4.32 velocity=46.875; origin xyz=-0.0259 -0.013 0 rpy=0 0 3.141592653589793 -> xyz=0 0.01415 0 rpy=0 0 0
- joint rear_right_hip_aa_joint: origin xyz=-0.10425 0.025 -0.02 rpy=0 0 0 -> xyz=-0.13424999999999998 0.025 -0.02 rpy=0 0 0
- joint rear_right_hip_fe_joint: limit lower=-0.17453292519943295 upper=0.7853981633974483 effort=4.45 velocity=47.125 -> lower=-0.7853981633974483 upper=0.17453292519943295 effort=2.43 velocity=83.33333333333333; origin xyz=0.0135 -0.0878 0 rpy=0 0 3.141592653589793 -> xyz=0.054678 -0.0878 0 rpy=0 0 0
- joint rear_right_lower_leg_joint: limit lower=-1.5707963267948966 upper=1.5707963267948966 effort=4.45 velocity=47.125 -> lower=-1.5707963267948966 upper=1.5707963267948966 effort=4.32 velocity=46.875; origin xyz=0 -0.0285 -0.134 rpy=0 0 0 -> xyz=0 -0.0315 -0.134 rpy=0 0 0
- joint rear_right_upper_leg_joint: limit lower=-1.5707963267948966 upper=1.5707963267948966 effort=4.45 velocity=47.125 -> lower=-1.5707963267948966 upper=1.5707963267948966 effort=4.32 velocity=46.875; origin xyz=-0.0259 0.013 0 rpy=0 0 3.141592653589793 -> xyz=0 -0.01415 0 rpy=0 0 0
- joint rear_spine_pitch_joint: limit lower=-0.2617993877991494 upper=0.2617993877991494 effort=4.45 velocity=47.125 -> lower=-0.2617993877991494 upper=0.2617993877991494 effort=4.32 velocity=46.875; origin xyz=-0.045 -0.025 -0.015 rpy=0 0 0 -> xyz=-0.045 0.0 -0.015 rpy=0 0 0
- joint rear_spine_yaw_joint: limit lower=-0.2617993877991494 upper=0.2617993877991494 effort=4.45 velocity=47.125 -> lower=-0.2617993877991494 upper=0.2617993877991494 effort=2.43 velocity=83.33333333333333; origin xyz=0 0.02505 0.02115 rpy=0 0 0 -> xyz=0 0 0.02115 rpy=0 0 0
